File: ADC_Breakout.kicad_pcb (KiCad board)
At the start: 2 copper layers, 55 x 55 mm, 67 parts, among them J0 Conn_01x06, J10 Conn_01x02, J11 Conn_01x02, J12 Conn_01x02, J13 Conn_01x02, J2 Digital Power, J3 Clock Chooser, J4 Analog Power, J6 Conn_01x02, J7 Conn_01x02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

Commit message: Layout updates
Parts:
- moved R1 3.67 mm to (148.8, 111.7)
- moved R2 2.04 mm to (151.0, 110.0)
Changed lines of the file:
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@@
 		(tags "capacitor")
 		(property "Reference" "C1"
-			(at 0 -1.68 90)
+			(at 2.375 0 180)
 			(layer "F.SilkS")
 			(effects
@@
 		(tags "capacitor")
 		(property "Reference" "C4"
-			(at 2.425 0.075 90)
+			(at 2.925 0 180)
 			(layer "F.SilkS")
 			(effects
@@
 		)
 		(property "Value" "1u"
-			(at 0 1.68 360)
+			(at 0 1.68 0)
 			(layer "F.Fab")
 			(effects
@@
 		)
 		(fp_text user "${REFERENCE}"
-			(at 0 0 360)
+			(at 0 0 0)
 			(layer "F.Fab")
 			(effects
@@
 	(footprint "Resistor_SMD:R_0805_2012Metric"
 		(layer "F.Cu")
-		(at 148.975 110.225 90)
+		(at 151 109.95 90)
 		(descr "Resistor SMD 0805 (2012 Metric), square (rectangular) end terminal, IPC_7351 nominal, (Body size source: IPC-SM-782 page 72, https://www.pcb-3d.com/wordpress/wp-content/uploads/ipc-sm-782a_amendment_1_and_2.pdf), generated with kicad-footprint-generator")
 		(tags "resistor")
 		(property "Reference" "R2"
-			(at 0 -1.65 90)
+			(at -2.45 -0.075 0)
 			(layer "F.SilkS")
 			(effects
@@
 	(footprint "Resistor_SMD:R_0805_2012Metric"
 		(layer "F.Cu")
-		(at 145.425 110.3875 -90)
+		(at 148.85 111.7 -90)
 		(descr "Resistor SMD 0805 (2012 Metric), square (rectangular) end terminal, IPC_7351 nominal, (Body size source: IPC-SM-782 page 72, https://www.pcb-3d.com/wordpress/wp-content/uploads/ipc-sm-782a_amendment_1_and_2.pdf), generated with kicad-footprint-generator")
 		(tags "resistor")
 		(property "Reference" "R1"
-			(at 0 1.5494 90)
+			(at -2.375 0.025 180)
 			(layer "F.SilkS")
 			(effects
@@
 		(tags "resistor")
 		(property "Reference" "R4"
-			(at -2.707999 -0.0239 90)
+			(at -2.5 -0.0239 180)
 			(layer "F.SilkS")
 			(effects
@@
 		(tags "resistor")
 		(property "Reference" "R3"
-			(at 0 -1.65 90)
+			(at 0 -1.95 180)
 			(layer "F.SilkS")
 			(effects
@@
 		(tags "Through hole pin header THT 1x02 2.54mm single row")
 		(property "Reference" "JP1"
-			(at 0 -2.33 360)
+			(at 0 -2.33 0)
 			(layer "F.SilkS")
 			(hide yes)
@@
 		)
 		(property "Value" "Jumper_2_Open"
-			(at 0 4.87 360)
+			(at 0 4.87 0)
 			(layer "F.Fab")
 			(effects
@@
 	)
 	(gr_text "DPWR"
-		(at 147.625 83.65 0)
+		(at 147.775 77.75 0)
 		(layer "F.SilkS")
 		(effects
@@
 	)
 	(gr_text "Disable\nClock"
-		(at 158.8 85.6 90)
+		(at 153.225 84.95 0)
 		(layer "F.SilkS")
 		(effects
@@
 				(thickness 0.153)
 			)
+			(justify right)
 		)
 	)
@@
 	)
 	(segment
-		(start 140.2875 115.8125)
-		(end 142.425 113.675)
+		(start 146.975 117.6625)
+		(end 145.125 115.8125)
 		(width 0.2)
 		(layer "B.Cu")
@@
 	)
 	(segment
-		(start 145.125 115.8125)
-		(end 140.2875 115.8125)
+		(start 140.2875 115.8125)
+		(end 142.425 113.675)
 		(width 0.2)
 		(layer "B.Cu")
@@
 	)
 	(segment
-		(start 146.975 117.6625)
-		(end 145.125 115.8125)
+		(start 145.125 115.8125)
+		(end 140.2875 115.8125)
 		(width 0.2)
 		(layer "B.Cu")
@@
 	)
 	(segment
-		(start 136.6368 102.894001)
-		(end 137.562299 102.894001)
-		(width 0.2)
-		(layer "F.Cu")
-		(net 27)
-	)
-	(segment
-		(start 141.659098 106.9908)
-		(end 151.9908 106.9908)
+		(start 137.562299 102.894001)
+		(end 141.659098 106.9908)
 		(width 0.2)
 		(layer "F.Cu")
@@
 	)
 	(segment
-		(start 151.9908 106.9908)
-		(end 154.1308 109.1308)
+		(start 136.6368 102.894001)
+		(end 137.562299 102.894001)
 		(width 0.2)
 		(layer "F.Cu")
@@
 	)
 	(segment
-		(start 137.562299 102.894001)
-		(end 141.659098 106.9908)
+		(start 141.659098 106.9908)
+		(end 153.8788 106.9908)
 		(width 0.2)
 		(layer "F.Cu")
@@
 	)
 	(segment
-		(start 154.1308 109.1308)
+		(start 153.8788 106.9908)
 		(end 156.0188 109.1308)
 		(width 0.2)
@@
 	)
 	(segment
-		(start 141.1147 108.275)
-		(end 147.9375 108.275)
+		(start 137.2337 104.394)
+		(end 141.1147 108.275)
 		(width 0.2)
 		(layer "F.Cu")
@@
 	)
 	(segment
-		(start 148.975 109.3125)
-		(end 152.2125 109.3125)
+		(start 154.2 114.932)
+		(end 156.0188 116.7508)
 		(width 0.2)
 		(layer "F.Cu")
@@
 	)
 	(segment
-		(start 147.9375 108.275)
-		(end 148.975 109.3125)
+		(start 141.1147 108.275)
+		(end 150.2375 108.275)
 		(width 0.2)
 		(layer "F.Cu")
@@
 	)
 	(segment
-		(start 154.2 114.932)
-		(end 156.0188 116.7508)
+		(start 151.275 109.3125)
+		(end 152.2125 109.3125)
 		(width 0.2)
 		(layer "F.Cu")
@@
 	)
 	(segment
-		(start 152.2125 109.3125)
-		(end 154.2 111.3)
+		(start 154.2 111.3)
+		(end 154.2 114.932)
 		(width 0.2)
 		(layer "F.Cu")
@@
 	)
 	(segment
-		(start 137.2337 104.394)
-		(end 141.1147 108.275)
+		(start 152.2125 109.3125)
+		(end 154.2 111.3)
 		(width 0.2)
 		(layer "F.Cu")
@@
 	)
 	(segment
-		(start 154.2 111.3)
-		(end 154.2 114.932)
+		(start 151 109.0375)
+		(end 151.275 109.3125)
 		(width 0.2)
 		(layer "F.Cu")
@@
 	)
 	(segment
+		(start 150.2375 108.275)
+		(end 151 109.0375)
+		(width 0.2)
+		(layer "F.Cu")
+		(net 31)
+	)
+	(segment
 		(start 155.325 89.4375)
 		(end 155.325 86.69)
@@
 	)
 	(segment
-		(start 150.025 112.95)
-		(end 150.75 113.675)
+		(start 148.85 112.6125)
+		(end 150.875 114.6375)
 		(width 0.2)
 		(layer "F.Cu")
@@
 	)
 	(segment
-		(start 145.425 111.3)
-		(end 147.075 112.95)
+		(start 150.875 120.002898)
+		(end 150.127899 120.749999)
 		(width 0.2)
 		(layer "F.Cu")
@@
 	)
 	(segment
-		(start 150.75 120.127898)
-		(end 150.127899 120.749999)
+		(start 150.127899 120.749999)
+		(end 150.127899 126.500001)
 		(width 0.2)
 		(layer "F.Cu")
@@
 	)
 	(segment
-		(start 140.641998 111.3)
-		(end 145.425 111.3)
+		(start 145.2125 112.6125)
+		(end 148.85 112.6125)
 		(width 0.2)
 		(layer "F.Cu")
@@
 	(segment
 		(start 135.186399 105.844401)
-		(end 140.641998 111.3)
+		(end 140.041998 110.7)
 		(width 0.2)
 		(layer "F.Cu")
@@
 	)
 	(segment
-		(start 150.75 113.675)
-		(end 150.75 120.127898)
+		(start 140.041998 110.7)
+		(end 143.3 110.7)
 		(width 0.2)
 		(layer "F.Cu")
@@
 	)
 	(segment
-		(start 150.127899 120.749999)
-		(end 150.127899 126.500001)
+		(start 150.875 114.6375)
+		(end 150.875 120.002898)
 		(width 0.2)
 		(layer "F.Cu")
@@
 	)
 	(segment
-		(start 147.075 112.95)
-		(end 150.025 112.95)
+		(start 143.3 110.7)
+		(end 145.2125 112.6125)
 		(width 0.2)
 		(layer "F.Cu")
@@
 			(thermal_gap 0.5)
 			(thermal_bridge_width 0.5)
-			(smoothing fillet)
-			(radius 1)
 		)
 		(polygon

Commit message: Added graphics + iBOM
Parts:
- added LOGO0: LHRs, Top:LHRs_LOGO, B.Cu at (125.5, 97.9)
- added LOGO1: UTSVT Logo, SVT_Special:UTSVT_Logo_Symbol, B.Cu at (125.9, 90.8)
- moved R6 10.0 mm to (150.9, 126.0), turned to 180 degrees
- moved D2 7.33 mm to (150.9, 123.8), turned to 180 degrees
- moved SW1 6.00 mm to (149.9, 118.0)
- moved TP4 3.53 mm to (140.7, 116.8)
- moved TP5 3.41 mm to (142.4, 113.8)
- moved R1 2.67 mm to (146.3, 111.0)
Routing:
- net /ADC/NSYNC: track 31.5 -> 23.3 mm
- net VDDA: track 36.3 -> 33.0 mm
- net /REFIN: track 28.2 -> 30.7 mm
- net GND: track 10.7 -> 8.86 mm
- net /INT_OSC: track 7.67 -> 6.15 mm
- net /CS: track 26.6 -> 25.6 mm
- net VDD: track 6.63 -> 5.86 mm
- net /A6_N: track 2.80 -> 2.26 mm
- net /A4_N: track 2.79 -> 2.26 mm
- net /A7_N: track 2.78 -> 2.24 mm
- net /A5_N: track 2.80 -> 2.27 mm
- net /A3_N: track 2.80 -> 2.27 mm
- net GNDA: track 45.6 -> 46.0 mm, vias 2 -> 1
Other:
- board text added: "ADS131M08-Q1 ADC Breakout Board v1 Shaun Kurian March 2025"
