File: ADC_Breakout.kicad_pcb (KiCad board)
At the start: 2 copper layers, 55 x 55 mm, 69 parts, among them J0 Conn_01x06, J10 Conn_01x02, J11 Conn_01x02, J12 Conn_01x02, J13 Conn_01x02, J2 Digital Power, J3 Clock Chooser, J4 Analog Power, J6 Conn_01x02, J7 Conn_01x02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

Commit message: gerebres
Parts:
- added JP0: AGND_JMP, Jumper:SolderJumper-2_P1.3mm_Open_TrianglePad1.0x1.5mm, B.Cu at (130.4, 85.5)
- added JP2: AGND_JMP, Jumper:SolderJumper-2_P1.3mm_Open_TrianglePad1.0x1.5mm, B.Cu at (124.7, 85.4)
- added JP3: AGND_JMP, Jumper:SolderJumper-2_P1.3mm_Open_TrianglePad1.0x1.5mm, B.Cu at (118.2, 91.1)
- added JP4: AGND_JMP, Jumper:SolderJumper-2_P1.3mm_Open_TrianglePad1.0x1.5mm, B.Cu at (118.2, 96.6)
- added JP5: AGND_JMP, Jumper:SolderJumper-2_P1.3mm_Open_TrianglePad1.0x1.5mm, B.Cu at (118.2, 107.2)
- added JP6: AGND_JMP, Jumper:SolderJumper-2_P1.3mm_Open_TrianglePad1.0x1.5mm, B.Cu at (118.2, 113.2)
- added JP7: AGND_JMP, Jumper:SolderJumper-2_P1.3mm_Open_TrianglePad1.0x1.5mm, B.Cu at (123.8, 119.9)
- added JP8: AGND_JMP, Jumper:SolderJumper-2_P1.3mm_Open_TrianglePad1.0x1.5mm, B.Cu at (130.3, 119.9)
- added R0: 100k, Resistor_SMD:R_0805_2012Metric, F.Cu at (156.0, 119.7)
- moved LOGO0 17.5 mm to (129.5, 115.0)
- moved LOGO1 5.10 mm to (131.0, 91.5)
- moved D2 2.67 mm to (148.3, 123.8)
- moved R6 2.67 mm to (148.3, 126.0)
- moved R1 1.83 mm to (144.4, 110.8), turned to 180 degrees
- moved R2 1.60 mm to (149.4, 109.8)
- turned C3 to 90 degrees
Routing:
- net GNDA: track 46.0 -> 11.8 mm
- net /CLKIN: track 5.53 -> 20.7 mm
- net /*DRDY: track 24.8 -> 31.4 mm
- net GND: track 8.86 -> 12.9 mm
- net /A5_N: track 2.27 -> 5.16 mm
- net /A7_N: track 2.24 -> 5.13 mm
- net /A6_N: track 2.26 -> 5.15 mm
- net /A0_N: track 2.41 -> 5.27 mm
- net /A2_N: track 2.40 -> 5.25 mm
- net /A4_N: track 2.26 -> 5.10 mm
- net /A1_N: track 2.39 -> 5.23 mm
- net /A3_N: track 2.27 -> 5.09 mm
- net VDDA: track 33.0 -> 32.1 mm
- net /ADC/FA2_P: track 17.4 -> 18.2 mm
- net /ADC/FA5_P: track 16.6 -> 17.4 mm
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- added copper zone on B.Cu, net GNDA
- added copper zone on F.Cu, net GNDA
- removed copper zone on F.Cu, net /CLKIN
