File: ADS131H08QPBSRQ1.kicad_sch (KiCad schematic)
At the start: 31 parts, among them U1 ADS131M08QPBSRQ1

Commit message: gerebres
Parts:
- added R0: 100k, Resistor_SMD:R_0805_2012Metric, symbol Device:R
Connections:
- net AGND is gone; now on net GNDA: U1.13 (AGND)
- net *DRDY: now also R0.2
- net VDD: now also R0.1
- net AVDD renamed VDDA
Other:
- moved on the sheet: R2
